File: Electronics/MCU.sch (EAGLE design)
At the start: 14 parts, among them IC2 74AC157D, J77 uart, U1 ATMEGA2560-16AU-TQFP100, U2 AT25DF041A-SH-B

Commit message: Add uart0 breakout
Parts:
- added C1, C2, C3, C4, C5, C6, C7, C8: (no value), rcl:C-EUC0805
- added JP9: FTDI_DEVICE, SparkFun-Connectors:FTDI_DEVICE
- added TP1: TEST-POINT3X5, SparkFun:TEST-POINT3X5
- added TP10, TP11, TP13, TP2, TP3, TP4, TP5, TP6, TP7, TP8, TP9: TEST-POINT2, SparkFun:TEST-POINT2
Connections:
- new net N$10: TP6.1, U1.PH5(OC4C)
- new net N$11: TP7.1, U1.PH4(OC4B)
- new net N$12: TP8.1, U1.(XCK0/AIN0)PE2
- new net N$13: TP9.1, U1.PH2(XCK2)
- new net N$14: TP10.1, U1.(OC3B/INT4)PE4
- new net N$15: TP11.1, U1.(OC3C/INT5)PE5
- new net N$17: TP13.1, U1.(OC3A/AIN1)PE3
- new net N$5: TP1.1, U1.PJ2(XCK3/PCINT11)
- new net N$6: TP2.1, U1.(TOSC2)PG3
- new net N$7: TP3.1, U1.(TOSC1)PG4
- new net N$8: TP4.1, U1.PH7(T4)
- new net N$9: TP5.1, U1.PH6(OC2B)
- new net RX2: JP9.RXI, U1.(RXD0/PCIN8)PE0
- new net TX2: JP9.TXO, U1.(TXD0)PE1
- net GND: now also C1.2, C2.2, C3.2, C4.2, C5.2, C6.2, C7.2, C8.2
- net HALT: now also U1.(ADC0)PF0; no longer U1.(OC3B/INT4)PE4
- net INT: now also U1.(ADC1)PF1; no longer U1.(OC3A/AIN1)PE3
- net VCC: now also C1.1, C2.1, C3.1, C4.1, C5.1, C6.1, C7.1, C8.1, U1.PJ3(PCINT12), U1.PJ4(PCINT13)
Changed lines of the file:
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@@
 <part name="J77" library="SparkFun" deviceset="M02" device="PTH" value="uart"/>
 <part name="UART1" library="SparkFun" deviceset="M02" device="PTH" value="i2c"/>
+<part name="C1" library="rcl" deviceset="C-EU" device="C0805"/>
+<part name="C2" library="rcl" deviceset="C-EU" device="C0805"/>
+<part name="C3" library="rcl" deviceset="C-EU" device="C0805"/>
+<part name="C4" library="rcl" deviceset="C-EU" device="C0805"/>
+<part name="C5" library="rcl" deviceset="C-EU" device="C0805"/>
+<part name="C6" library="rcl" deviceset="C-EU" device="C0805"/>
+<part name="TP1" library="SparkFun" deviceset="TEST-POINT" device="3X5"/>
+<part name="TP2" library="SparkFun" deviceset="TEST-POINT" device="2"/>
+<part name="TP3" library="SparkFun" deviceset="TEST-POINT" device="2"/>
+<part name="TP4" library="SparkFun" deviceset="TEST-POINT" device="2"/>
+<part name="TP5" library="SparkFun" deviceset="TEST-POINT" device="2"/>
+<part name="TP6" library="SparkFun" deviceset="TEST-POINT" device="2"/>
+<part name="TP7" library="SparkFun" deviceset="TEST-POINT" device="2"/>
+<part name="TP9" library="SparkFun" deviceset="TEST-POINT" device="2"/>
+<part name="TP8" library="SparkFun" deviceset="TEST-POINT" device="2"/>
+<part name="TP11" library="SparkFun" deviceset="TEST-POINT" device="2"/>
+<part name="C7" library="rcl" deviceset="C-EU" device="C0805"/>
+<part name="C8" library="rcl" deviceset="C-EU" device="C0805"/>
+<part name="JP9" library="SparkFun-Connectors" deviceset="FTDI_DEVICE" device=""/>
+<part name="TP10" library="SparkFun" deviceset="TEST-POINT" device="2"/>
+<part name="TP13" library="SparkFun" deviceset="TEST-POINT" device="2"/>
 </parts>
 <sheets>
@@
 <instance part="J77" gate="G$1" x="22.86" y="-66.04"/>
 <instance part="UART1" gate="G$1" x="109.22" y="0" rot="R180"/>
+<instance part="C1" gate="G$1" x="129.54" y="93.98"/>
+<instance part="C2" gate="G$1" x="134.62" y="93.98"/>
+<instance part="C3" gate="G$1" x="139.7" y="93.98"/>
+<instance part="C4" gate="G$1" x="144.78" y="93.98"/>
+<instance part="C5" gate="G$1" x="149.86" y="93.98"/>
+<instance part="C6" gate="G$1" x="154.94" y="93.98"/>
+<instance part="TP1" gate="G$1" x="30.48" y="-38.1" rot="R180"/>
+<instance part="TP2" gate="G$1" x="101.6" y="-58.42"/>
+<instance part="TP3" gate="G$1" x="101.6" y="-55.88"/>
+<instance part="TP4" gate="G$1" x="30.48" y="-48.26" rot="R180"/>
+<instance part="TP5" gate="G$1" x="30.48" y="-50.8" rot="R180"/>
+<instance part="TP6" gate="G$1" x="30.48" y="-53.34" rot="R180"/>
+<instance part="TP7" gate="G$1" x="30.48" y="-55.88" rot="R180"/>
+<instance part="TP9" gate="G$1" x="30.48" y="-60.96" rot="R180"/>
+<instance part="TP8" gate="G$1" x="101.6" y="-20.32"/>
+<instance part="TP11" gate="G$1" x="101.6" y="-12.7"/>
+<instance part="C7" gate="G$1" x="160.02" y="93.98"/>
+<instance part="C8" gate="G$1" x="165.1" y="93.98"/>
+<instance part="JP9" gate="G$1" x="170.18" y="-10.16"/>
+<instance part="TP10" gate="G$1" x="101.6" y="-15.24"/>
+<instance part="TP13" gate="G$1" x="101.6" y="-17.78"/>
 </instances>
 <busses>
@@
 <junction x="25.4" y="66.04"/>
 </segment>
+<segment>
+<pinref part="C1" gate="G$1" pin="1"/>
+<pinref part="C2" gate="G$1" pin="1"/>
+<junction x="149.86" y="96.52"/>
+<pinref part="C3" gate="G$1" pin="1"/>
+<pinref part="C4" gate="G$1" pin="1"/>
+<junction x="139.7" y="96.52"/>
+<wire x1="129.54" y1="96.52" x2="124.46" y2="96.52" width="0.1524" layer="91"/>
+<wire x1="144.78" y1="96.52" x2="139.7" y2="96.52" width="0.1524" layer="91"/>
+<wire x1="139.7" y1="96.52" x2="134.62" y2="96.52" width="0.1524" layer="91"/>
+<junction x="134.62" y="96.52"/>
+<wire x1="134.62" y1="96.52" x2="129.54" y2="96.52" width="0.1524" layer="91"/>
+<pinref part="C5" gate="G$1" pin="1"/>
+<pinref part="C6" gate="G$1" pin="1"/>
+<wire x1="149.86" y1="96.52" x2="160.02" y2="96.52" width="0.1524" layer="91"/>
+<junction x="165.1" y="96.52"/>
+<junction x="144.78" y="96.52"/>
+<junction x="129.54" y="96.52"/>
+<pinref part="C7" gate="G$1" pin="1"/>
+<pinref part="C8" gate="G$1" pin="1"/>
+<wire x1="160.02" y1="96.52" x2="144.78" y2="96.52" width="0.1524" layer="91"/>
+<wire x1="165.1" y1="96.52" x2="160.02" y2="96.52" width="0.1524" layer="91"/>
+<junction x="160.02" y="96.52"/>
+<wire x1="160.02" y1="96.52" x2="154.94" y2="96.52" width="0.1524" layer="91"/>
+</segment>
+<segment>
+<pinref part="U1" gate="1" pin="PJ3(PCINT12)"/>
+<wire x1="30.48" y1="-35.56" x2="-7.62" y2="-35.56" width="0.1524" layer="91"/>
+<label x="17.78" y="-35.56" size="1.778" layer="95"/>
+</segment>
+<segment>
+<pinref part="U1" gate="1" pin="PJ4(PCINT13)"/>
+<wire x1="30.48" y1="-33.02" x2="-7.62" y2="-33.02" width="0.1524" layer="91"/>
+<label x="17.78" y="-33.02" size="1.778" layer="95"/>
+</segment>
 </net>
 <net name="GND" class="0">
@@
 <wire x1="30.48" y1="63.5" x2="-7.62" y2="63.5" width="0.1524" layer="91"/>
 </segment>
+<segment>
+<pinref part="C1" gate="G$1" pin="2"/>
+<pinref part="C2" gate="G$1" pin="2"/>
+<junction x="149.86" y="88.9"/>
+<pinref part="C3" gate="G$1" pin="2"/>
+<pinref part="C4" gate="G$1" pin="2"/>
+<junction x="139.7" y="88.9"/>
+<wire x1="129.54" y1="88.9" x2="124.46" y2="88.9" width="0.1524" layer="91"/>
+<wire x1="144.78" y1="88.9" x2="139.7" y2="88.9" width="0.1524" layer="91"/>
+<wire x1="139.7" y1="88.9" x2="134.62" y2="88.9" width="0.1524" layer="91"/>
+<junction x="134.62" y="88.9"/>
+<wire x1="134.62" y1="88.9" x2="129.54" y2="88.9" width="0.1524" layer="91"/>
+<pinref part="C5" gate="G$1" pin="2"/>
+<pinref part="C6" gate="G$1" pin="2"/>
+<wire x1="149.86" y1="88.9" x2="160.02" y2="88.9" width="0.1524" layer="91"/>
+<junction x="165.1" y="88.9"/>
+<junction x="144.78" y="88.9"/>
+<junction x="129.54" y="88.9"/>
+<pinref part="C7" gate="G$1" pin="2"/>
+<pinref part="C8" gate="G$1" pin="2"/>
+<wire x1="160.02" y1="88.9" x2="144.78" y2="88.9" width="0.1524" layer="91"/>
+<wire x1="165.1" y1="88.9" x2="160.02" y2="88.9" width="0.1524" layer="91"/>
+<junction x="160.02" y="88.9"/>
+<wire x1="160.02" y1="88.9" x2="154.94" y2="88.9" width="0.1524" layer="91"/>
+</segment>
 </net>
 <net name="WR" class="0">
@@
 </segment>
 <segment>
-<pinref part="U1" gate="1" pin="(OC3B/INT4)PE4"/>
-<wire x1="124.46" y1="-15.24" x2="101.6" y2="-15.24" width="0.1524" layer="91"/>
+<pinref part="U1" gate="1" pin="(ADC0)PF0"/>
+<wire x1="124.46" y1="-48.26" x2="101.6" y2="-48.26" width="0.1524" layer="91"/>
+<label x="109.22" y="-48.26" size="1.778" layer="95"/>
 </segment>
 </net>
@@
 </segment>
 <segment>
-<pinref part="U1" gate="1" pin="(OC3A/AIN1)PE3"/>
-<wire x1="124.46" y1="-17.78" x2="101.6" y2="-17.78" width="0.1524" layer="91"/>
+<pinref part="U1" gate="1" pin="(ADC1)PF1"/>
+<wire x1="124.46" y1="-45.72" x2="101.6" y2="-45.72" width="0.1524" layer="91"/>
+<label x="109.22" y="-45.72" size="1.778" layer="95"/>
 </segment>
 </net>
@@
 </segment>
 </net>
+<net name="N$5" class="0">
+<segment>
+<pinref part="U1" gate="1" pin="PJ2(XCK3/PCINT11)"/>
+<pinref part="TP1" gate="G$1" pin="1"/>
+</segment>
+</net>
+<net name="N$6" class="0">
+<segment>
+<pinref part="U1" gate="1" pin="(TOSC2)PG3"/>
+<pinref part="TP2" gate="G$1" pin="1"/>
+</segment>
+</net>
+<net name="N$7" class="0">
+<segment>
+<pinref part="U1" gate="1" pin="(TOSC1)PG4"/>
+<pinref part="TP3" gate="G$1" pin="1"/>
+</segment>
+</net>
+<net name="N$8" class="0">
+<segment>
+<pinref part="U1" gate="1" pin="PH7(T4)"/>
+<pinref part="TP4" gate="G$1" pin="1"/>
+</segment>
+</net>
+<net name="N$9" class="0">
+<segment>
+<pinref part="U1" gate="1" pin="PH6(OC2B)"/>
+<pinref part="TP5" gate="G$1" pin="1"/>
+</segment>
+</net>
+<net name="N$10" class="0">
+<segment>
+<pinref part="U1" gate="1" pin="PH5(OC4C)"/>
+<pinref part="TP6" gate="G$1" pin="1"/>
+</segment>
+</net>
+<net name="N$11" class="0">
+<segment>
+<pinref part="U1" gate="1" pin="PH4(OC4B)"/>
+<pinref part="TP7" gate="G$1" pin="1"/>
+</segment>
+</net>
+<net name="N$13" class="0">
+<segment>
+<pinref part="U1" gate="1" pin="PH2(XCK2)"/>
+<pinref part="TP9" gate="G$1" pin="1"/>
+</segment>
+</net>
+<net name="N$12" class="0">
+<segment>
+<pinref part="U1" gate="1" pin="(XCK0/AIN0)PE2"/>
+<pinref part="TP8" gate="G$1" pin="1"/>
+</segment>
+</net>
+<net name="N$15" class="0">
+<segment>
+<pinref part="U1" gate="1" pin="(OC3C/INT5)PE5"/>
+<pinref part="TP11" gate="G$1" pin="1"/>
+</segment>
+</net>
+<net name="TX2" class="0">
+<segment>
+<pinref part="JP9" gate="G$1" pin="TXO"/>
+<wire x1="165.1" y1="-7.62" x2="162.56" y2="-7.62" width="0.1524" layer="91"/>
+<label x="162.56" y="-7.62" size="1.778" layer="95"/>
+</segment>
+<segment>
+<pinref part="U1" gate="1" pin="(TXD0)PE1"/>
+<wire x1="101.6" y1="-22.86" x2="104.14" y2="-22.86" width="0.1524" layer="91"/>
+</segment>
+</net>
+<net name="RX2" class="0">
+<segment>
+<pinref part="JP9" gate="G$1" pin="RXI"/>
+<wire x1="165.1" y1="-10.16" x2="162.56" y2="-10.16" width="0.1524" layer="91"/>
+<label x="162.56" y="-10.16" size="1.778" layer="95"/>
+</segment>
+<segment>
+<pinref part="U1" gate="1" pin="(RXD0/PCIN8)PE0"/>
+<wire x1="101.6" y1="-25.4" x2="104.14" y2="-25.4" width="0.1524" layer="91"/>
+</segment>
+</net>
+<net name="N$14" class="0">
+<segment>
+<pinref part="U1" gate="1" pin="(OC3B/INT4)PE4"/>
+<pinref part="TP10" gate="G$1" pin="1"/>
+</segment>
+</net>
+<net name="N$17" class="0">
+<segment>
+<pinref part="U1" gate="1" pin="(OC3A/AIN1)PE3"/>
+<pinref part="TP13" gate="G$1" pin="1"/>
+</segment>
+</net>

Commit message: Layout changes
Connections:
- net GND: now also IC2A.G
Changed lines of the file:
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@@
 <part name="TP10" library="SparkFun" deviceset="TEST-POINT" device="2"/>
 <part name="TP13" library="SparkFun" deviceset="TEST-POINT" device="2"/>
+<part name="GND5" library="SparkFun" deviceset="GND" device=""/>
 </parts>
 <sheets>
@@
 <instance part="TP10" gate="G$1" x="101.6" y="-15.24"/>
 <instance part="TP13" gate="G$1" x="101.6" y="-17.78"/>
+<instance part="GND5" gate="1" x="142.24" y="-93.98"/>
 </instances>
 <busses>
@@
 <wire x1="160.02" y1="88.9" x2="154.94" y2="88.9" width="0.1524" layer="91"/>
 </segment>
-</net>
+<segment>
+<pinref part="IC2" gate="A" pin="G"/>
+<pinref part="GND5" gate="1" pin="GND"/>
+</segment>
+</net>

Commit message: Fix up caps on ram/mcu board
Parts:
- added C9: (no value), rcl:C-EUC0805
- added TP12: TEST-POINT2, SparkFun:TEST-POINT2
Connections:
- new net N$16: C9.2, JP9.DTR
- net /RESET: now also C9.1, U1.RESET
- net CLKO: now also TP12.1
- net GND: now also JP9.GND
- net IORQ: now also U1.(TXD1/INT3)PD3; no longer U1.(XCK1)PD5
- net MREQ: now also U1.(RXD1/INT2)PD2; no longer U1.(ICP1)PD4
- net RESET: now also U1.(XCK1)PD5; no longer U1.(TXD1/INT3)PD3
- net VCC: now also JP9.VCC
Changed lines of the file:
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@@
 <part name="TP13" library="SparkFun" deviceset="TEST-POINT" device="2"/>
 <part name="GND5" library="SparkFun" deviceset="GND" device=""/>
+<part name="GND6" library="SparkFun" deviceset="GND" device=""/>
+<part name="P+12" library="SparkFun" deviceset="VCC" device=""/>
+<part name="C9" library="rcl" deviceset="C-EU" device="C0805"/>
+<part name="TP12" library="SparkFun" deviceset="TEST-POINT" device="2"/>
 </parts>
 <sheets>
@@
 <instance part="TP13" gate="G$1" x="101.6" y="-17.78"/>
 <instance part="GND5" gate="1" x="142.24" y="-93.98"/>
+<instance part="GND6" gate="1" x="165.1" y="-20.32"/>
+<instance part="P+12" gate="1" x="165.1" y="-12.7" rot="R90"/>
+<instance part="C9" gate="G$1" x="165.1" y="0"/>
+<instance part="TP12" gate="G$1" x="137.16" y="-66.04" rot="R90"/>
 </instances>
 <busses>
@@
 <label x="17.78" y="-33.02" size="1.778" layer="95"/>
 </segment>
+<segment>
+<pinref part="JP9" gate="G$1" pin="VCC"/>
+<pinref part="P+12" gate="1" pin="VCC"/>
+</segment>
 </net>
 <net name="GND" class="0">
@@
 <pinref part="GND5" gate="1" pin="GND"/>
 </segment>
+<segment>
+<pinref part="JP9" gate="G$1" pin="GND"/>
+<pinref part="GND6" gate="1" pin="GND"/>
+</segment>
 </net>
 <net name="WR" class="0">
@@
 <pinref part="U1" gate="1" pin="(T0)PD7"/>
 <wire x1="124.46" y1="15.24" x2="101.6" y2="15.24" width="0.1524" layer="91"/>
+<label x="104.14" y="15.24" size="1.778" layer="95"/>
 </segment>
 </net>
@@
 <pinref part="U1" gate="1" pin="(T1)PD6"/>
 <wire x1="124.46" y1="12.7" x2="101.6" y2="12.7" width="0.1524" layer="91"/>
+<label x="104.14" y="12.7" size="1.778" layer="95"/>
 </segment>
 </net>
@@
 </segment>
 <segment>
-<pinref part="U1" gate="1" pin="(XCK1)PD5"/>
-<wire x1="124.46" y1="10.16" x2="101.6" y2="10.16" width="0.1524" layer="91"/>
+<pinref part="U1" gate="1" pin="(TXD1/INT3)PD3"/>
+<wire x1="124.46" y1="5.08" x2="101.6" y2="5.08" width="0.1524" layer="91"/>
+<label x="104.14" y="5.08" size="1.778" layer="95"/>
 </segment>
 </net>
@@
 </segment>
 <segment>
-<pinref part="U1" gate="1" pin="(ICP1)PD4"/>
-<wire x1="124.46" y1="7.62" x2="101.6" y2="7.62" width="0.1524" layer="91"/>
+<pinref part="U1" gate="1" pin="(RXD1/INT2)PD2"/>
+<wire x1="101.6" y1="2.54" x2="124.46" y2="2.54" width="0.1524" layer="91"/>
+<label x="104.14" y="2.54" size="1.778" layer="95"/>
 </segment>
 </net>
@@
 </segment>
 <segment>
-<pinref part="U1" gate="1" pin="(TXD1/INT3)PD3"/>
-<wire x1="124.46" y1="5.08" x2="101.6" y2="5.08" width="0.1524" layer="91"/>
+<pinref part="U1" gate="1" pin="(XCK1)PD5"/>
+<wire x1="124.46" y1="10.16" x2="101.6" y2="10.16" width="0.1524" layer="91"/>
+<label x="104.14" y="10.16" size="1.778" layer="95"/>
 </segment>
 </net>
@@
 <label x="157.48" y="-38.1" size="1.778" layer="95"/>
 </segment>
+<segment>
+<pinref part="U1" gate="1" pin="RESET"/>
+<wire x1="30.48" y1="83.82" x2="25.4" y2="83.82" width="0.1524" layer="91"/>
+<label x="15.24" y="83.82" size="1.778" layer="95"/>
+</segment>
+<segment>
+<pinref part="C9" gate="G$1" pin="1"/>
+<wire x1="165.1" y1="2.54" x2="170.18" y2="2.54" width="0.1524" layer="91"/>
+</segment>
 </net>
 <net name="TDO" class="0">
@@
 <wire x1="142.24" y1="-66.04" x2="137.16" y2="-66.04" width="0.1524" layer="91"/>
 <label x="134.62" y="-66.04" size="1.778" layer="95"/>
+<pinref part="TP12" gate="G$1" pin="1"/>
 </segment>
 </net>
@@
 </segment>
 </net>
+<net name="N$16" class="0">
+<segment>
+<pinref part="JP9" gate="G$1" pin="DTR"/>
+<pinref part="C9" gate="G$1" pin="2"/>
+</segment>
+</net>
